File: Omni_Trigger.sch (KiCad schematic (older format))
At the start: 43 parts, among them J1 Screw_Terminal_01x02, J2 Screw_Terminal_01x02, J3 Conn_02x13_Top_Bottom, J4 Conn_02x04_Odd_Even, J5 Conn_02x02_Odd_Even, J6 Conn_02x04_Odd_Even, J7 Screw_Terminal_01x08, J8 Screw_Terminal_01x04, K1 G5LE-1, K2 G5LE-1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

Commit message: Updated clearances
Parts:
- XA1: symbol arduino:Arduino_Nano_Socket -> Omni_Trigger-rescue:Arduino_Nano_Socket-arduino
Changed lines of the file:
@@
 $EndDescr
 $Comp
-L arduino:Arduino_Nano_Socket XA1
+L Omni_Trigger-rescue:Arduino_Nano_Socket-arduino XA1
 U 1 1 5F628F8B
 P 4200 3300
